File: Microcontroller.sch (KiCad schematic (older format))
At the start: 17 parts, among them P3 USB_B, P5 JTAG, U5 ATMEGA32U4RC-A, Y1 12MHz

Commit message: Layout
Parts:
- added C30: 1µF, Capacitors_SMD:C_0805_HandSoldering, symbol C
- C23, C24, C25, C26, C27: footprint Capacitors_SMD:C_0603_HandSoldering -> Capacitors_SMD:C_0805_HandSoldering
- P3: footprint Connect:USB_B -> w_conn_pc:conn_usb_B_mini_smd
- Y1: footprint Crystals:Crystal_HC49-SD_SMD -> w_crystal:hc-49_smd
Connections:
- net GND: now also C30.2
- net VCC: now also C30.1
- net C_IO5: no longer names the net of U5.26 ((T1/~OC4D~/ADC9)PD6)
- net C_IO6: no longer names the net of U5.27 ((T0/OC4D/ADC10)PD7)
- net Clock_Out: no longer names the net of U5.32 ((ICP3/CLK0/OC4A)PC7)
- no-connect marks 5 -> 8
Changed lines of the file:
@@
 LIBS:switches
 LIBS:xo-14s
+LIBS:oscillator_xo
 LIBS:FPGABoard-cache
 EELAYER 25 0
@@
 F 0 "P3" H 1950 3450 50  0000 C CNN
 F 1 "USB_B" H 1700 3850 50  0000 C CNN
-F 2 "Connect:USB_B" V 1700 3550 50  0001 C CNN
+F 2 "w_conn_pc:conn_usb_B_mini_smd" V 1700 3550 50  0001 C CNN
 F 3 "" V 1700 3550 50  0000 C CNN
 	1    1750 3650
@@
 F 0 "Y1" H 2950 2850 50  0000 C CNN
 F 1 "12MHz" H 2950 2650 50  0000 C CNN
-F 2 "Crystals:Crystal_HC49-SD_SMD" H 2950 2750 50  0001 C CNN
+F 2 "w_crystal:hc-49_smd" H 2950 2750 50  0001 C CNN
 F 3 "" H 2950 2750 50  0000 C CNN
 	1    2950 2750
@@
 CS_C
 $Comp
-L GND #PWR028
+L GND #PWR030
 U 1 1 577EB04B
 P 4150 5550
-F 0 "#PWR028" H 4150 5300 50  0001 C CNN
+F 0 "#PWR030" H 4150 5300 50  0001 C CNN
 F 1 "GND" H 4150 5400 50  0000 C CNN
 F 2 "" H 4150 5550 50  0000 C CNN
@@
 $EndComp
 $Comp
-L GND #PWR029
+L GND #PWR031
 U 1 1 577EB215
 P 2100 3900
-F 0 "#PWR029" H 2100 3650 50  0001 C CNN
+F 0 "#PWR031" H 2100 3650 50  0001 C CNN
 F 1 "GND" H 2100 3750 50  0000 C CNN
 F 2 "" H 2100 3900 50  0000 C CNN
@@
 $EndComp
 $Comp
-L GND #PWR030
+L GND #PWR032
 U 1 1 577EB26B
 P 1650 4050
-F 0 "#PWR030" H 1650 3800 50  0001 C CNN
+F 0 "#PWR032" H 1650 3800 50  0001 C CNN
 F 1 "GND" H 1650 3900 50  0000 C CNN
 F 2 "" H 1650 4050 50  0000 C CNN
@@
 F 0 "C27" H 2960 3020 50  0000 L CNN
 F 1 "22pF" H 2960 2870 50  0000 L CNN
-F 2 "Capacitors_SMD:C_0603_HandSoldering" H 2950 2950 50  0001 C CNN
+F 2 "Capacitors_SMD:C_0805_HandSoldering" H 2950 2950 50  0001 C CNN
 F 3 "" H 2950 2950 50  0000 C CNN
 	1    2950 2950
@@
 F 0 "C26" H 2610 3020 50  0000 L CNN
 F 1 "22pF" H 2610 2870 50  0000 L CNN
-F 2 "Capacitors_SMD:C_0603_HandSoldering" H 2600 2950 50  0001 C CNN
+F 2 "Capacitors_SMD:C_0805_HandSoldering" H 2600 2950 50  0001 C CNN
 F 3 "" H 2600 2950 50  0000 C CNN
 	1    2600 2950
@@
 $EndComp
 $Comp
-L GND #PWR031
+L GND #PWR033
 U 1 1 5780F9B3
 P 2800 3100
-F 0 "#PWR031" H 2800 2850 50  0001 C CNN
+F 0 "#PWR033" H 2800 2850 50  0001 C CNN
 F 1 "GND" H 2800 2950 50  0000 C CNN
 F 2 "" H 2800 3100 50  0000 C CNN
@@
 $EndComp
 $Comp
-L GND #PWR032
+L GND #PWR034
 U 1 1 5780FD97
 P 2950 4250
-F 0 "#PWR032" H 2950 4000 50  0001 C CNN
+F 0 "#PWR034" H 2950 4000 50  0001 C CNN
 F 1 "GND" H 2950 4100 50  0000 C CNN
 F 2 "" H 2950 4250 50  0000 C CNN
@@
 $EndComp
 $Comp
-L GND #PWR033
+L GND #PWR035
 U 1 1 57812B8C
 P 8050 5350
-F 0 "#PWR033" H 8050 5100 50  0001 C CNN
+F 0 "#PWR035" H 8050 5100 50  0001 C CNN
 F 1 "GND" H 8050 5200 50  0000 C CNN
 F 2 "" H 8050 5350 50  0000 C CNN
@@
 F 0 "C23" H 2675 7000 50  0000 L CNN
 F 1 "100nF" H 2675 6800 50  0000 L CNN
-F 2 "Capacitors_SMD:C_0603_HandSoldering" H 2688 6750 50  0001 C CNN
+F 2 "Capacitors_SMD:C_0805_HandSoldering" H 2688 6750 50  0001 C CNN
 F 3 "" H 2650 6900 50  0000 C CNN
 	1    2650 6900
@@
 F 0 "C24" H 2975 7000 50  0000 L CNN
 F 1 "100nF" H 2975 6800 50  0000 L CNN
-F 2 "Capacitors_SMD:C_0603_HandSoldering" H 2988 6750 50  0001 C CNN
+F 2 "Capacitors_SMD:C_0805_HandSoldering" H 2988 6750 50  0001 C CNN
 F 3 "" H 2950 6900 50  0000 C CNN
 	1    2950 6900
@@
 F 0 "C25" H 3275 7000 50  0000 L CNN
 F 1 "100nF" H 3275 6800 50  0000 L CNN
-F 2 "Capacitors_SMD:C_0603_HandSoldering" H 3288 6750 50  0001 C CNN
+F 2 "Capacitors_SMD:C_0805_HandSoldering" H 3288 6750 50  0001 C CNN
 F 3 "" H 3250 6900 50  0000 C CNN
 	1    3250 6900
@@
 $EndComp
 $Comp
-L GND #PWR034
+L GND #PWR036
 U 1 1 57817BBC
 P 2800 7150
-F 0 "#PWR034" H 2800 6900 50  0001 C CNN
+F 0 "#PWR036" H 2800 6900 50  0001 C CNN
 F 1 "GND" H 2800 7000 50  0000 C CNN
 F 2 "" H 2800 7150 50  0000 C CNN
@@
 	2800 6650 2800 6600
 Wire Wire Line
-	2350 6650 3250 6650
+	2100 6650 3250 6650
 Wire Wire Line
 	2350 6650 2350 6750
@@
 	2350 7050 2350 7100
 Wire Wire Line
-	2350 7100 3250 7100
+	2100 7100 3250 7100
 Wire Wire Line
 	2800 7100 2800 7150
@@
 $EndComp
 $Comp
-L GND #PWR035
+L GND #PWR037
 U 1 1 5781915B
 P 5600 6100
-F 0 "#PWR035" H 5600 5850 50  0001 C CNN
+F 0 "#PWR037" H 5600 5850 50  0001 C CNN
 F 1 "GND" H 5600 5950 50  0000 C CNN
 F 2 "" H 5600 6100 50  0000 C CNN
@@
 Text HLabel 5800 2850 2    60   Input ~ 0
 INIT_B
-Text Label 7350 1400 0    60   ~ 0
+Text Label 8150 5050 0    60   ~ 0
 RESET
 Wire Wire Line
@@
 Wire Wire Line
 	5300 2850 5800 2850
-Text HLabel 5800 3250 2    60   Output ~ 0
-Clock_Out
 NoConn ~ 5300 3650
-Text HLabel 6800 4350 2    60   BiDi ~ 0
-C_IO[1..6]
+Text HLabel 6750 4050 2    60   BiDi ~ 0
+C_IO[1..4]
 Wire Bus Line
-	6650 3250 6650 4350
+	6650 3250 6650 4050
 Wire Bus Line
-	6650 3550 6650 4250
-Wire Bus Line
-	6650 3650 6650 4150
+	6650 3550 6650 3950
 Entry Wire Line
 	6550 3450 6650 3550
@@
 Entry Wire Line
 	6550 3850 6650 3950
-Entry Wire Line
-	6550 4050 6650 4150
-Entry Wire Line
-	6550 4150 6650 4250
 Wire Wire Line
 	5300 3150 6550 3150
 Wire Wire Line
 	5300 3850 6550 3850
-Wire Wire Line
-	5300 4050 6550 4050
-Wire Wire Line
-	5300 4150 6550 4150
-Wire Wire Line
-	5300 3250 5800 3250
 Wire Bus Line
-	6650 4350 6800 4350
-Wire Wire Line
-	2900 1400 7350 1400
-Wire Wire Line
-	7350 1400 7350 4150
-Wire Wire Line
-	7350 4150 8150 4150
-Wire Wire Line
-	8150 4150 8150 5050
+	6650 4050 6750 4050
+Wire Wire Line
+	2900 1400 8150 1400
+Wire Wire Line
+	8150 1400 8150 5050
 NoConn ~ 5300 2950
 $Comp
-L VCC #PWR036
+L VCC #PWR038
 U 1 1 57871A81
 P 4200 1800
-F 0 "#PWR036" H 4200 1650 50  0001 C CNN
+F 0 "#PWR038" H 4200 1650 50  0001 C CNN
 F 1 "VCC" H 4200 1950 50  0000 C CNN
 F 2 "" H 4200 1800 50  0000 C CNN
@@
 $EndComp
 $Comp
-L VCC #PWR037
+L VCC #PWR039
 U 1 1 57871EAB
 P 8000 4600
-F 0 "#PWR037" H 8000 4450 50  0001 C CNN
+F 0 "#PWR039" H 8000 4450 50  0001 C CNN
 F 1 "VCC" H 8000 4750 50  0000 C CNN
 F 2 "" H 8000 4600 50  0000 C CNN
@@
 $EndComp
 $Comp
-L VCC #PWR038
+L VCC #PWR040
 U 1 1 578720B7
 P 2800 6600
-F 0 "#PWR038" H 2800 6450 50  0001 C CNN
+F 0 "#PWR040" H 2800 6450 50  0001 C CNN
 F 1 "VCC" H 2800 6750 50  0000 C CNN
 F 2 "" H 2800 6600 50  0000 C CNN
@@
 Text Label 6300 3850 0    60   ~ 0
 C_IO4
-Text Label 6300 4050 0    60   ~ 0
-C_IO5
-Text Label 6300 4150 0    60   ~ 0
-C_IO6
 Wire Wire Line
 	5300 2450 5800 2450
@@
 Text Label 2100 3650 0    60   ~ 0
 DC+
+$Comp
+L C C30
+U 1 1 578ECA14
+P 2100 6900
+F 0 "C30" H 2125 7000 50  0000 L CNN
+F 1 "1µF" H 2125 6800 50  0000 L CNN
+F 2 "Capacitors_SMD:C_0805_HandSoldering" H 2138 6750 50  0001 C CNN
+F 3 "" H 2100 6900 50  0000 C CNN
+	1    2100 6900
+	1    0    0    -1
+$EndComp
+Wire Wire Line
+	2100 6650 2100 6750
+Connection ~ 2350 6650
+Wire Wire Line
+	2100 7100 2100 7050
+Connection ~ 2350 7100
+NoConn ~ 5300 3250
+NoConn ~ 5300 4150
+NoConn ~ 5300 4050
 $EndSCHEMATC

Commit message: Additional Caps at VCC, Layout
Parts:
- C23, C24, C25, C26, C27: footprint Capacitors_SMD:C_0805_HandSoldering -> Capacitors_SMD:C_0603_HandSoldering
Changed lines of the file:
@@
 F 0 "C27" H 2960 3020 50  0000 L CNN
 F 1 "22pF" H 2960 2870 50  0000 L CNN
-F 2 "Capacitors_SMD:C_0805_HandSoldering" H 2950 2950 50  0001 C CNN
+F 2 "Capacitors_SMD:C_0603_HandSoldering" H 2950 2950 50  0001 C CNN
 F 3 "" H 2950 2950 50  0000 C CNN
 	1    2950 2950
@@
 F 0 "C26" H 2610 3020 50  0000 L CNN
 F 1 "22pF" H 2610 2870 50  0000 L CNN
-F 2 "Capacitors_SMD:C_0805_HandSoldering" H 2600 2950 50  0001 C CNN
+F 2 "Capacitors_SMD:C_0603_HandSoldering" H 2600 2950 50  0001 C CNN
 F 3 "" H 2600 2950 50  0000 C CNN
 	1    2600 2950
@@
 F 0 "C23" H 2675 7000 50  0000 L CNN
 F 1 "100nF" H 2675 6800 50  0000 L CNN
-F 2 "Capacitors_SMD:C_0805_HandSoldering" H 2688 6750 50  0001 C CNN
+F 2 "Capacitors_SMD:C_0603_HandSoldering" H 2688 6750 50  0001 C CNN
 F 3 "" H 2650 6900 50  0000 C CNN
 	1    2650 6900
@@
 F 0 "C24" H 2975 7000 50  0000 L CNN
 F 1 "100nF" H 2975 6800 50  0000 L CNN
-F 2 "Capacitors_SMD:C_0805_HandSoldering" H 2988 6750 50  0001 C CNN
+F 2 "Capacitors_SMD:C_0603_HandSoldering" H 2988 6750 50  0001 C CNN
 F 3 "" H 2950 6900 50  0000 C CNN
 	1    2950 6900
@@
 F 0 "C25" H 3275 7000 50  0000 L CNN
 F 1 "100nF" H 3275 6800 50  0000 L CNN
-F 2 "Capacitors_SMD:C_0805_HandSoldering" H 3288 6750 50  0001 C CNN
+F 2 "Capacitors_SMD:C_0603_HandSoldering" H 3288 6750 50  0001 C CNN
 F 3 "" H 3250 6900 50  0000 C CNN
 	1    3250 6900
@@
 	1    0    0    -1
 $EndComp
-Wire Wire Line
-	2100 6650 2100 6750
 Connection ~ 2350 6650
-Wire Wire Line
-	2100 7100 2100 7050
 Connection ~ 2350 7100
 NoConn ~ 5300 3250
 NoConn ~ 5300 4150
 NoConn ~ 5300 4050
+Wire Wire Line
+	2100 6650 2100 6750
+Wire Wire Line
+	2100 7100 2100 7050
 $EndSCHEMATC
