File: Connections.sch (KiCad schematic (older format))
At the start: 18 parts, among them P4 CONN_02X07, P6 CONN_02X07, P7 CONN_02X07, P8 CONN_02X07, SW1 SW_PUSH, SW2 SW_PUSH

Commit message: Release for Manufacture
Parts:
- SW1, SW2: footprint SMD_Switch_LSX1301:SW_LSx_1301 -> Buttons_Switches_SMD:SW_SPST_B3S-1000
Changed lines of the file:
@@
 F 0 "SW1" H 7100 1860 50  0000 C CNN
 F 1 "SW_PUSH" H 6950 1670 50  0000 C CNN
-F 2 "SMD_Switch_LSX1301:SW_LSx_1301" H 6950 1750 50  0001 C CNN
+F 2 "Buttons_Switches_SMD:SW_SPST_B3S-1000" H 6950 1750 50  0001 C CNN
 F 3 "" H 6950 1750 50  0000 C CNN
 	1    6950 1750
@@
 F 0 "SW2" H 7100 2260 50  0000 C CNN
 F 1 "SW_PUSH" H 6950 2070 50  0000 C CNN
-F 2 "SMD_Switch_LSX1301:SW_LSx_1301" H 6950 2150 50  0001 C CNN
+F 2 "Buttons_Switches_SMD:SW_SPST_B3S-1000" H 6950 2150 50  0001 C CNN
 F 3 "" H 6950 2150 50  0000 C CNN
 	1    6950 2150
@@
 $EndComp
 $Comp
-L GND #PWR46
+L GND #PWR045
 U 1 1 5782F652
 P 4450 2300
-F 0 "#PWR46" H 4450 2050 50  0001 C CNN
+F 0 "#PWR045" H 4450 2050 50  0001 C CNN
 F 1 "GND" H 4450 2150 50  0000 C CNN
 F 2 "" H 4450 2300 50  0000 C CNN
@@
 LED3
 $Comp
-L GND #PWR45
+L GND #PWR046
 U 1 1 5782FC2F
 P 7500 2250
-F 0 "#PWR45" H 7500 2000 50  0001 C CNN
+F 0 "#PWR046" H 7500 2000 50  0001 C CNN
 F 1 "GND" H 7500 2100 50  0000 C CNN
 F 2 "" H 7500 2250 50  0000 C CNN
@@
 GPIO0[1..12]
 $Comp
-L GND #PWR50
+L GND #PWR047
 U 1 1 5784BCA2
 P 4650 3450
-F 0 "#PWR50" H 4650 3200 50  0001 C CNN
+F 0 "#PWR047" H 4650 3200 50  0001 C CNN
 F 1 "GND" H 4650 3300 50  0000 C CNN
 F 2 "" H 4650 3450 50  0000 C CNN
@@
 GPIO1[1..12]
 $Comp
-L GND #PWR54
+L GND #PWR048
 U 1 1 5785BA09
 P 4750 5150
-F 0 "#PWR54" H 4750 4900 50  0001 C CNN
+F 0 "#PWR048" H 4750 4900 50  0001 C CNN
 F 1 "GND" H 4750 5000 50  0000 C CNN
 F 2 "" H 4750 5150 50  0000 C CNN
@@
 GPIO2[1..12]
 $Comp
-L GND #PWR56
+L GND #PWR049
 U 1 1 5785C545
 P 4750 5550
-F 0 "#PWR56" H 4750 5300 50  0001 C CNN
+F 0 "#PWR049" H 4750 5300 50  0001 C CNN
 F 1 "GND" H 4750 5400 50  0000 C CNN
 F 2 "" H 4750 5550 50  0000 C CNN
@@
 GPIO36
 $Comp
-L GND #PWR51
+L GND #PWR050
 U 1 1 57864245
 P 7400 3450
-F 0 "#PWR51" H 7400 3200 50  0001 C CNN
+F 0 "#PWR050" H 7400 3200 50  0001 C CNN
 F 1 "GND" H 7400 3300 50  0000 C CNN
 F 2 "" H 7400 3450 50  0000 C CNN
@@
 $EndComp
 $Comp
-L VCC #PWR48
+L VCC #PWR051
 U 1 1 57871160
 P 3550 3350
-F 0 "#PWR48" H 3550 3200 50  0001 C CNN
+F 0 "#PWR051" H 3550 3200 50  0001 C CNN
 F 1 "VCC" H 3550 3500 50  0000 C CNN
 F 2 "" H 3550 3350 50  0000 C CNN
@@
 $EndComp
 $Comp
-L VCC #PWR47
+L VCC #PWR052
 U 1 1 578714DD
 P 6300 3250
-F 0 "#PWR47" H 6300 3100 50  0001 C CNN
+F 0 "#PWR052" H 6300 3100 50  0001 C CNN
 F 1 "VCC" H 6300 3400 50  0000 C CNN
 F 2 "" H 6300 3250 50  0000 C CNN
@@
 $EndComp
 $Comp
-L VCC #PWR53
+L VCC #PWR053
 U 1 1 57871512
 P 3550 4450
-F 0 "#PWR53" H 3550 4300 50  0001 C CNN
+F 0 "#PWR053" H 3550 4300 50  0001 C CNN
 F 1 "VCC" H 3550 4600 50  0000 C CNN
 F 2 "" H 3550 4450 50  0000 C CNN
@@
 $EndComp
 $Comp
-L VCC #PWR55
+L VCC #PWR054
 U 1 1 57871547
 P 3550 5450
-F 0 "#PWR55" H 3550 5300 50  0001 C CNN
+F 0 "#PWR054" H 3550 5300 50  0001 C CNN
 F 1 "VCC" H 3550 5600 50  0000 C CNN
 F 2 "" H 3550 5450 50  0000 C CNN
@@
 Connection ~ 6500 2150
 $Comp
-L VCC #PWR44
+L VCC #PWR055
 U 1 1 58AE5184
 P 6400 1250
-F 0 "#PWR44" H 6400 1100 50  0001 C CNN
+F 0 "#PWR055" H 6400 1100 50  0001 C CNN
 F 1 "VCC" H 6400 1400 50  0000 C CNN
 F 2 "" H 6400 1250 50  0000 C CNN
@@
 $EndComp
 $Comp
-L VCC #PWR49
+L VCC #PWR056
 U 1 1 58AE572C
 P 1600 3400
-F 0 "#PWR49" H 1600 3250 50  0001 C CNN
+F 0 "#PWR056" H 1600 3250 50  0001 C CNN
 F 1 "VCC" H 1600 3550 50  0000 C CNN
 F 2 "" H 1600 3400 50  0000 C CNN
@@
 $EndComp
 $Comp
-L GND #PWR52
+L GND #PWR057
 U 1 1 58AE5764
 P 1600 3900
-F 0 "#PWR52" H 1600 3650 50  0001 C CNN
+F 0 "#PWR057" H 1600 3650 50  0001 C CNN
 F 1 "GND" H 1600 3750 50  0000 C CNN
 F 2 "" H 1600 3900 50  0000 C CNN
