File: Spartan3A.sch (KiCad schematic (older format))
At the start: 37 parts, among them P1 JTAG_FPGA, Q1 BSS123, SW3 SW_Push, SW4 SW_DIP_x02, U1 XC3S50A/VQ100, U6 M25P20, U7 XO53

Commit message: Release for Manufacture
Parts:
- SW3: footprint SMD_Switch_LSX1301:SW_LSx_1301 -> Buttons_Switches_SMD:SW_SPST_B3S-1000
Changed lines of the file:
@@
 $EndComp
 $Comp
-L GND #PWR2
+L GND #PWR01
 U 1 1 5748F443
 P 4100 2800
-F 0 "#PWR2" H 4100 2550 50  0001 C CNN
+F 0 "#PWR01" H 4100 2550 50  0001 C CNN
 F 1 "GND" H 4100 2650 50  0000 C CNN
 F 2 "" H 4100 2800 50  0000 C CNN
@@
 NoConn ~ 4700 2750
 $Comp
-L GND #PWR16
+L GND #PWR02
 U 1 1 5748F44F
 P 8200 7850
-F 0 "#PWR16" H 8200 7600 50  0001 C CNN
+F 0 "#PWR02" H 8200 7600 50  0001 C CNN
 F 1 "GND" H 8200 7700 50  0000 C CNN
 F 2 "" H 8200 7850 50  0000 C CNN
@@
 $EndComp
 $Comp
-L GND #PWR23
+L GND #PWR03
 U 1 1 5748F4A8
 P 9850 10400
-F 0 "#PWR23" H 9850 10150 50  0001 C CNN
+F 0 "#PWR03" H 9850 10150 50  0001 C CNN
 F 1 "GND" H 9850 10250 50  0000 C CNN
 F 2 "" H 9850 10400 50  0000 C CNN
@@
 $EndComp
 $Comp
-L GND #PWR22
+L GND #PWR04
 U 1 1 5748F4C4
 P 8500 10400
-F 0 "#PWR22" H 8500 10150 50  0001 C CNN
+F 0 "#PWR04" H 8500 10150 50  0001 C CNN
 F 1 "GND" H 8500 10250 50  0000 C CNN
 F 2 "" H 8500 10400 50  0000 C CNN
@@
 $EndComp
 $Comp
-L GND #PWR21
+L GND #PWR05
 U 1 1 5748F4E6
 P 6800 10400
-F 0 "#PWR21" H 6800 10150 50  0001 C CNN
+F 0 "#PWR05" H 6800 10150 50  0001 C CNN
 F 1 "GND" H 6800 10250 50  0000 C CNN
 F 2 "" H 6800 10400 50  0000 C CNN
@@
 	10600 4100 10700 4200
 $Comp
-L GND #PWR6
+L GND #PWR06
 U 1 1 57828260
 P 12700 4950
-F 0 "#PWR6" H 12700 4700 50  0001 C CNN
+F 0 "#PWR06" H 12700 4700 50  0001 C CNN
 F 1 "GND" H 12700 4800 50  0000 C CNN
 F 2 "" H 12700 4950 50  0000 C CNN
@@
 $EndComp
 $Comp
-L GND #PWR14
+L GND #PWR07
 U 1 1 57830E2E
 P 2850 7550
-F 0 "#PWR14" H 2850 7300 50  0001 C CNN
+F 0 "#PWR07" H 2850 7300 50  0001 C CNN
 F 1 "GND" H 2850 7400 50  0000 C CNN
 F 2 "" H 2850 7550 50  0000 C CNN
@@
 $EndComp
 $Comp
-L GND #PWR15
+L GND #PWR08
 U 1 1 578324A6
 P 3850 7550
-F 0 "#PWR15" H 3850 7300 50  0001 C CNN
+F 0 "#PWR08" H 3850 7300 50  0001 C CNN
 F 1 "GND" H 3850 7400 50  0000 C CNN
 F 2 "" H 3850 7550 50  0000 C CNN
@@
 CS_FPGA
 $Comp
-L GND #PWR5
+L GND #PWR09
 U 1 1 5748F50A
 P 2400 4300
-F 0 "#PWR5" H 2400 4050 50  0001 C CNN
+F 0 "#PWR09" H 2400 4050 50  0001 C CNN
 F 1 "GND" H 2400 4150 50  0000 C CNN
 F 2 "" H 2400 4300 50  0000 C CNN
@@
 $EndComp
 $Comp
-L GND #PWR20
+L GND #PWR010
 U 1 1 5783F7F7
 P 1850 10300
-F 0 "#PWR20" H 1850 10050 50  0001 C CNN
+F 0 "#PWR010" H 1850 10050 50  0001 C CNN
 F 1 "GND" H 1850 10150 50  0000 C CNN
 F 2 "" H 1850 10300 50  0000 C CNN
@@
 DONE
 $Comp
-L VCC #PWR1
+L VCC #PWR011
 U 1 1 5786CFE3
 P 7950 2000
-F 0 "#PWR1" H 7950 1850 50  0001 C CNN
+F 0 "#PWR011" H 7950 1850 50  0001 C CNN
 F 1 "VCC" H 7950 2150 50  0000 C CNN
 F 2 "" H 7950 2000 50  0000 C CNN
@@
 VCC_AUX
 $Comp
-L VCC #PWR11
+L VCC #PWR012
 U 1 1 5786E3E9
 P 3850 6750
-F 0 "#PWR11" H 3850 6600 50  0001 C CNN
+F 0 "#PWR012" H 3850 6600 50  0001 C CNN
 F 1 "VCC" H 3850 6900 50  0000 C CNN
 F 2 "" H 3850 6750 50  0000 C CNN
@@
 $EndComp
 $Comp
-L VCC #PWR10
+L VCC #PWR013
 U 1 1 5786E437
 P 2850 6700
-F 0 "#PWR10" H 2850 6550 50  0001 C CNN
+F 0 "#PWR013" H 2850 6550 50  0001 C CNN
 F 1 "VCC" H 2850 6850 50  0000 C CNN
 F 2 "" H 2850 6700 50  0000 C CNN
@@
 $EndComp
 $Comp
-L VCC #PWR17
+L VCC #PWR014
 U 1 1 5786E6C9
 P 1850 8800
-F 0 "#PWR17" H 1850 8650 50  0001 C CNN
+F 0 "#PWR014" H 1850 8650 50  0001 C CNN
 F 1 "VCC" H 1850 8950 50  0000 C CNN
 F 2 "" H 1850 8800 50  0000 C CNN
@@
 $EndComp
 $Comp
-L VCC #PWR18
+L VCC #PWR015
 U 1 1 5786EDEE
 P 6800 9650
-F 0 "#PWR18" H 6800 9500 50  0001 C CNN
+F 0 "#PWR015" H 6800 9500 50  0001 C CNN
 F 1 "VCC" H 6800 9800 50  0000 C CNN
 F 2 "" H 6800 9650 50  0000 C CNN
@@
 VCC_INT
 $Comp
-L VCC #PWR3
+L VCC #PWR016
 U 1 1 5787091E
 P 2400 3550
-F 0 "#PWR3" H 2400 3400 50  0001 C CNN
+F 0 "#PWR016" H 2400 3400 50  0001 C CNN
 F 1 "VCC" H 2400 3700 50  0000 C CNN
 F 2 "" H 2400 3550 50  0000 C CNN
@@
 F 0 "SW3" H 3000 10100 50  0000 L CNN
 F 1 "SW_Push" H 2950 9940 50  0000 C CNN
-F 2 "SMD_Switch_LSX1301:SW_LSx_1301" H 2950 10200 50  0001 C CNN
+F 2 "Buttons_Switches_SMD:SW_SPST_B3S-1000" H 2950 10200 50  0001 C CNN
 F 3 "" H 2950 10200 50  0000 C CNN
 	1    2950 10000
@@
 $EndComp
 $Comp
-L GND #PWR19
+L GND #PWR017
 U 1 1 58B11500
 P 3250 10050
-F 0 "#PWR19" H 3250 9800 50  0001 C CNN
+F 0 "#PWR017" H 3250 9800 50  0001 C CNN
 F 1 "GND" H 3250 9900 50  0000 C CNN
 F 2 "" H 3250 10050 50  0000 C CNN
@@
 $EndComp
 $Comp
-L VCC #PWR4
+L VCC #PWR018
 U 1 1 58BA93EC
 P 13775 3675
-F 0 "#PWR4" H 13775 3525 50  0001 C CNN
+F 0 "#PWR018" H 13775 3525 50  0001 C CNN
 F 1 "VCC" H 13775 3825 50  0000 C CNN
 F 2 "" H 13775 3675 50  0000 C CNN
@@
 $EndComp
 $Comp
-L VCC #PWR9
+L VCC #PWR019
 U 1 1 58BA9730
 P 13700 6025
-F 0 "#PWR9" H 13700 5875 50  0001 C CNN
+F 0 "#PWR019" H 13700 5875 50  0001 C CNN
 F 1 "VCC" H 13700 6175 50  0000 C CNN
 F 2 "" H 13700 6025 50  0000 C CNN
@@
 $EndComp
 $Comp
-L GND #PWR12
+L GND #PWR020
 U 1 1 58BABD21
 P 13100 7375
-F 0 "#PWR12" H 13100 7125 50  0001 C CNN
+F 0 "#PWR020" H 13100 7125 50  0001 C CNN
 F 1 "GND" H 13100 7225 50  0000 C CNN
 F 2 "" H 13100 7375 50  0000 C CNN
@@
 $EndComp
 $Comp
-L GND #PWR7
+L GND #PWR021
 U 1 1 58BAC5DE
 P 13100 4975
-F 0 "#PWR7" H 13100 4725 50  0001 C CNN
+F 0 "#PWR021" H 13100 4725 50  0001 C CNN
 F 1 "GND" H 13100 4825 50  0000 C CNN
 F 2 "" H 13100 4975 50  0000 C CNN
@@
 $EndComp
 $Comp
-L GND #PWR8
+L GND #PWR022
 U 1 1 58BAC907
 P 14350 5025
-F 0 "#PWR8" H 14350 4775 50  0001 C CNN
+F 0 "#PWR022" H 14350 4775 50  0001 C CNN
 F 1 "GND" H 14350 4875 50  0000 C CNN
 F 2 "" H 14350 5025 50  0000 C CNN
@@
 Connection ~ 14300 6850
 $Comp
-L GND #PWR13
+L GND #PWR023
 U 1 1 58BADEB6
 P 14300 7375
-F 0 "#PWR13" H 14300 7125 50  0001 C CNN
+F 0 "#PWR023" H 14300 7125 50  0001 C CNN
 F 1 "GND" H 14300 7225 50  0000 C CNN
 F 2 "" H 14300 7375 50  0000 C CNN
